File: hardware/power-monitor.kicad_pcb (KiCad board)
At the start: 2 copper layers, 60 x 48 mm, 43 parts, among them J1 Screw_Terminal_01x02, J2 Screw_Terminal_01x02, J3 Screw_Terminal_01x02, J6 PROG, Q3 Q_NMOS_GSD, SW3 RESET, U1 INA228, U2 INA228, U3 LM74700, U4 LMR51610XDBVR, U5 ESP32-C3-WROOM-02-NOTHERMAL

Commit message: rev 1
Parts:
- removed the C3 at (173.9, 104.3)
- removed the J3 at (150.0, 110.0)
- removed NT1, NT2, NT3, NT4: NetTie_2, footprints:NetTie-2_SMD_Pad0.25mm
- removed Q3: Q_NMOS_GSD, Package_TO_SOT_SMD:TSOT-23_HandSoldering
- removed the R7 at (157.0, 102.5)
- removed the U3 at (172.9, 99.2)
- added C5: 0.1uF, Capacitor_SMD:C_0603_1608Metric_Pad1.08x0.95mm_HandSolder, F.Cu at (161.2, 76.4)
- added J10: I2C, Connector_JST:JST_SH_SM04B-SRSS-TB_1x04-1MP_P1.00mm_Horizontal, F.Cu at (147.5, 106.5)
- added J4: Output, TerminalBlock_Wuerth:Wuerth_REDCUBE-THR_WP-THRSH_74651175_THR, F.Cu at (142.0, 75.0)
- added J5: Screw_Terminal_01x01, TerminalBlock_Wuerth:Wuerth_REDCUBE-THR_WP-THRSH_74651175_THR, F.Cu at (178.0, 74.0)
- added J6: Ground, TerminalBlock_Wuerth:Wuerth_REDCUBE-THR_WP-THRSH_74651175_THR, F.Cu at (178.0, 85.0)
- added J7: Input B, TerminalBlock_Wuerth:Wuerth_REDCUBE-THR_WP-THRSH_74651175_THR, F.Cu at (142.0, 95.0)
- added J8: Screw_Terminal_01x01, TerminalBlock_Wuerth:Wuerth_REDCUBE-THR_WP-THRSH_74651175_THR, F.Cu at (178.0, 96.0)
- added J9: I2C, Connector_JST:JST_PH_S4B-PH-SM4-TB_1x04-1MP_P2.00mm_Horizontal, F.Cu at (160.0, 104.8)
- added R3: 2mOhm, Resistor_SMD:R_2816_7142Metric_Pad3.20x4.45mm_HandSolder, F.Cu at (142.0, 65.0)
- C3: renamed from C1; footprint Capacitor_SMD:C_1206_3216Metric_Pad1.33x1.80mm_HandSolder -> Capacitor_SMD:C_0603_1608Metric_Pad1.08x0.95mm_HandSolder
- C7: renamed from C5; footprint Capacitor_SMD:C_1206_3216Metric_Pad1.33x1.80mm_HandSolder -> Capacitor_SMD:C_0603_1608Metric_Pad1.08x0.95mm_HandSolder
- C8: renamed from C6; footprint Capacitor_SMD:C_1210_3225Metric_Pad1.33x2.70mm_HandSolder -> Capacitor_SMD:C_1206_3216Metric_Pad1.33x1.80mm_HandSolder
- C9: renamed from C2; footprint Capacitor_SMD:C_1206_3216Metric_Pad1.33x1.80mm_HandSolder -> Capacitor_SMD:C_0603_1608Metric_Pad1.08x0.95mm_HandSolder
- J1: value Screw_Terminal_01x02 -> Input A; footprint TerminalBlock_Phoenix:TerminalBlock_Phoenix_PT-1,5-2-5.0-H_1x02_P5.00mm_Horizontal -> TerminalBlock_Wuerth:Wuerth_REDCUBE-THR_WP-THRSH_74651175_THR
- J2: value Screw_Terminal_01x02 -> Screw_Terminal_01x06; footprint TerminalBlock_Phoenix:TerminalBlock_Phoenix_PT-1,5-2-5.0-H_1x02_P5.00mm_Horizontal -> TerminalBlock_Phoenix:TerminalBlock_Phoenix_MPT-0,5-6-2.54_1x06_P2.54mm_Horizontal
- moved H1 70.7 mm to (139.0, 43.5), turned to -90 degrees
- moved H2 63.9 mm to (181.0, 43.5), turned to -90 degrees
- moved J1 55.1 mm to (142.0, 55.0), turned to -90 degrees
- moved SW1 52.1 mm to (172.5, 106.2)
- moved J2 51.8 mm to (181.0, 62.0), turned to 90 degrees
- moved D2 47.6 mm to (146.0, 42.8), turned to 90 degrees
- moved D1 47.4 mm to (143.2, 42.8), turned to 90 degrees
- moved R2 43.1 mm to (148.8, 42.8), turned to 90 degrees
- moved R1 39.4 mm to (151.5, 42.8), turned to 90 degrees
- moved H3 38.5 mm to (138.5, 106.5), turned to -90 degrees
- moved J3 36.9 mm to (170.4, 65.5), turned to 90 degrees
- moved H4 35.3 mm to (181.0, 106.5), turned to -90 degrees
- moved C3 33.2 mm to (147.0, 62.9), turned to 90 degrees
- moved R7 32.8 mm to (163.8, 64.5)
- moved U2 32.1 mm to (151.0, 64.2), turned to 180 degrees
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- renumbered C10 to C1, C9 to C2, C8 to C4, C4 to C6, D2 to D1, D1 to D2, H4 to H1, H1 to H2, H2 to H4, J6 to J3, R4 to R1, R2 to R10, R9 to R11, R6 to R12, R3 to R2, R10 to R4, R14 to R5, R13 to R6, R12 to R7, R1 to R8, R8 to R9, SW3 to SW1, U5 to U1, U1 to U2, U4 to U3, U2 to U4
Connections:
- net /ESP32/BOOT renamed /BOOT
- net /ESP32/EN renamed /EN
- net /ESP32/IO2 renamed /IO2
- net /ESP32/IO8 renamed /IO8
- net /ESP32/RXD renamed /RXD
- net /ESP32/SCL renamed /SCL
- net /ESP32/TXD renamed /TXD
- C6 pad 1: Net-(Q3-D) -> /VPOS
- J1 pad 1: /Sense1/INB -> Net-(J1-Pin_1)
- J2 pad 1: /Sense2/INA -> GND
- J2 pad 2: GND -> VCC
- R1 pad 1: Net-(U5-GPIO0/ADC1_CH0/XTAL_32K_P) -> /LED1
- R12 pad 1: /VPOS -> Net-(J7-Pin_1)
- R12 pad 2: /Sense1/INB -> /VPOS
- R2 pad 1: Net-(U5-GPIO1/ADC1_CH1/XTAL_32K_N) -> /LED2
- R8 pad 2: /ESP32/SDA -> /SDA
- U1 pad 10: unconnected-(U5-GPIO10-Pad10) -> /EXT3
- U1 pad 15: unconnected-(U5-GPIO3/ADC1_CH3-Pad15) -> /EXT2
- U1 pad 17: Net-(U5-GPIO1/ADC1_CH1/XTAL_32K_N) -> /EXT1
- U1 pad 18: Net-(U5-GPIO0/ADC1_CH0/XTAL_32K_P) -> /EXT0
- U1 pad 3: unconnected-(U5-GPIO4/ADC1_CH4-Pad3) -> /LED1
- U1 pad 4: unconnected-(U5-GPIO5/ADC2_CH0-Pad4) -> /LED2
- U1 pad 5: /ESP32/SDA -> /SDA
- U2 pad 10: Net-(U1-Vin+) -> /VPOS
- U2 pad 4: /ESP32/SDA -> /SDA
- U2 pad 8: Net-(U1-Vbus) -> Net-(J1-Pin_1)
- U2 pad 9: Net-(U1-Vbus) -> Net-(J1-Pin_1)
- U3 pad 4: Net-(Q3-D) -> /VPOS
- U3 pad 5: Net-(Q3-D) -> /VPOS
- U4 pad 1: VCC -> /SDA
- U4 pad 10: Net-(U2-Vin+) -> Net-(J7-Pin_1)
- U4 pad 2: VCC -> /SDA
- U4 pad 4: /ESP32/SDA -> /SDA
- U4 pad 8: Net-(U2-Vbus) -> Net-(J7-Pin_1)
- U4 pad 9: Net-(U2-Vbus) -> /VPOS
Routing:
- net /SDA: track 0.00 -> 78.3 mm
- net /EN: track 35.9 -> 82.5 mm, vias 0 -> 4
- net /SCL: track 30.6 -> 76.5 mm, vias 2 -> 0
- net VCC: track 115.6 -> 160.1 mm, vias 4 -> 2
- net /VPOS: track 0.00 -> 33.3 mm, vias 6 -> 1
- net /ESP32/SDA: track 32.7 -> 0.00 mm
- net /RXD: track 39.7 -> 7.93 mm, vias 2 -> 0
- net /TXD: track 37.8 -> 10.4 mm, vias 2 -> 0
- net /LED2: track 0.00 -> 13.9 mm, vias 0 -> 2
- net Net-(J7-Pin_1): track 0.00 -> 11.8 mm
- net /IO2: track 3.77 -> 14.6 mm
- net /EXT3: track 0.00 -> 10.5 mm
- net /LED1: track 0.00 -> 10.5 mm, vias 0 -> 2
- net /EXT1: track 0.00 -> 10.2 mm
- net /EXT2: track 0.00 -> 9.97 mm
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- added copper zone on F.Cu, net Net-(J1-Pin_1)
- added copper zone on F.Cu, net Net-(J7-Pin_1)
- removed copper zone on F.Cu, net /Sense1/INB
- removed copper zone on F.Cu, net /Sense2/INA
- removed copper zone on B.Cu, net /VPOS
- removed copper zone on F.Cu, net Net-(Q3-D)
Other:
- board size 60 x 48 mm -> 50 x 70 mm
- board text added: "Calan Mai Solar panel monitor rev 1 April 2024"
- board text added: "EXT0"
- board text added: "EXT1"
- board text added: "EXT2"
- board text added: "EXT3"
- board text added: "GND"
- board text added: "VCC"
- board text removed: "Calan Mai Solar panel monitor rev 1 Feb 2024"

Commit message: Improve BOM
Parts:
- C4: value C -> 1uF
- C7: value 0.1uF / 16V -> 0.1uF
- C8: value 22uF / 16V -> 10uF
- J1: value Input A -> ~
- J10, J9: value I2C -> ~
- J3: value PROG -> ~
- J4: value Output -> ~
- J5, J8: value Screw_Terminal_01x01 -> ~
- J6: value Ground -> ~
- J7: value Input B -> ~
Changed lines of the file:
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@@
 			)
 		)
-		(property "Value" "C"
+		(property "Value" "1uF"
 			(at 0 1.85 90)
 			(layer "F.Fab")
@@
 		(sheetname "Root")
 		(sheetfile "power-monitor.kicad_sch")
-		(attr exclude_from_pos_files)
+		(attr exclude_from_pos_files exclude_from_bom)
 		(fp_circle
 			(center 0 0)
@@
 			)
 		)
-		(property "Value" "I2C"
+		(property "Value" "~"
 			(at 0 -4.25 0)
 			(layer "F.SilkS")
+			(hide yes)
 			(effects
 				(font
@@
 			)
 		)
+		(property "Label" "I2C"
+			(at 0 -4.25 0)
+			(unlocked yes)
+			(layer "F.SilkS")
+			(effects
+				(font
+					(size 1 1)
+					(thickness 0.15)
+				)
+			)
+		)
 		(property ki_fp_filters "Connector*:*_1x??-1MP*")
 		(sheetname "Root")
@@
 		(sheetname "Root")
 		(sheetfile "power-monitor.kicad_sch")
-		(attr exclude_from_pos_files)
+		(attr exclude_from_pos_files exclude_from_bom)
 		(fp_circle
 			(center 0 0)
@@
 			)
 		)
-		(property "Value" "Screw_Terminal_01x01"
+		(property "Value" "~"
 			(at 0 6 0)
 			(layer "F.Fab")
@@
 		(tags "screw terminal thread redcube thr power connector")
 		(property "Reference" "J1"
-			(at 0 -6 270)
+			(at 0 -6 90)
 			(layer "F.SilkS")
 			(hide yes)
@@
 			)
 		)
-		(property "Value" "Input A"
+		(property "Value" "~"
 			(at 0 6 -90)
 			(unlocked yes)
 			(layer "F.SilkS")
+			(hide yes)
 			(effects
 				(font
@@
 			)
 		)
+		(property "Label" "Input A"
+			(at 0 6 -90)
+			(unlocked yes)
+			(layer "F.SilkS")
+			(hide yes)
+			(effects
+				(font
+					(size 1 1)
+					(thickness 0.15)
+				)
+			)
+		)
 		(property ki_fp_filters "TerminalBlock*:*")
 		(sheetname "Root")
@@
 		)
 		(fp_text user "${REFERENCE}"
-			(at 0 0 -90)
+			(at 0 0 90)
 			(layer "F.Fab")
 			(effects
@@
 			)
 		)
-		(property "Value" "Ground"
+		(property "Value" "~"
 			(at 6 0 90)
-			(layer "F.SilkS")
+			(layer "F.Fab")
+			(hide yes)
 			(effects
 				(font
@@
 			)
 		)
+		(property "Label" "Ground"
+			(at 6 0 90)
+			(unlocked yes)
+			(layer "F.SilkS")
+			(effects
+				(font
+					(size 1 1)
+					(thickness 0.15)
+				)
+			)
+		)
 		(property ki_fp_filters "TerminalBlock*:*")
 		(sheetname "Root")
@@
 			)
 		)
-		(property "Value" "Input B"
+		(property "Value" "~"
 			(at 0 6 -90)
 			(unlocked yes)
 			(layer "F.SilkS")
+			(hide yes)
 			(effects
 				(font
@@
 			)
 		)
+		(property "Label" "Input B"
+			(at 0 6 -90)
+			(unlocked yes)
+			(layer "F.SilkS")
+			(effects
+				(font
+					(size 1 1)
+					(thickness 0.15)
+				)
+			)
+		)
 		(property ki_fp_filters "TerminalBlock*:*")
 		(sheetname "Root")
@@
 		)
 		(fp_text user "${REFERENCE}"
-			(at 0 0 -90)
+			(at 0 0 90)
 			(layer "F.Fab")
 			(effects
@@
 			)
 		)
+		(property "Characteristics" "100V"
+			(at 0 0 90)
+			(unlocked yes)
+			(layer "F.Fab")
+			(hide yes)
+			(effects
+				(font
+					(size 1 1)
+					(thickness 0.15)
+				)
+			)
+		)
 		(property ki_fp_filters "C_*")
 		(sheetname "Supply")
@@
 			)
 		)
-		(property "Value" "22uF / 16V"
+		(property "Value" "10uF"
 			(at 0 1.85 90)
 			(layer "F.Fab")
@@
 			)
 		)
+		(property "Characteristics" "16V"
+			(at 0 0 90)
+			(unlocked yes)
+			(layer "F.Fab")
+			(hide yes)
+			(effects
+				(font
+					(size 1 1)
+					(thickness 0.15)
+				)
+			)
+		)
 		(property ki_fp_filters "C_*")
 		(sheetname "Supply")
@@
 			)
 		)
+		(property "Characteristics" "100V"
+			(at 0 0 90)
+			(unlocked yes)
+			(layer "F.Fab")
+			(hide yes)
+			(effects
+				(font
+					(size 1 1)
+					(thickness 0.15)
+				)
+			)
+		)
 		(property ki_fp_filters "C_*")
 		(sheetname "Supply")
@@
 			)
 		)
-		(property "Value" "0.1uF / 16V"
+		(property "Value" "0.1uF"
 			(at 0 1.43 180)
 			(layer "F.Fab")
@@
 			)
 		)
+		(property "Characteristics" "16V"
+			(at 0 0 180)
+			(unlocked yes)
+			(layer "F.Fab")
+			(hide yes)
+			(effects
+				(font
+					(size 1 1)
+					(thickness 0.15)
+				)
+			)
+		)
 		(property ki_fp_filters "C_*")
 		(sheetname "Supply")
@@
 		(sheetname "Root")
 		(sheetfile "power-monitor.kicad_sch")
-		(attr exclude_from_pos_files)
+		(attr exclude_from_pos_files exclude_from_bom)
 		(fp_circle
 			(center 0 0)
@@
 			)
 		)
-		(property "Value" "Screw_Terminal_01x01"
+		(property "Value" "~"
 			(at 0 6 0)
 			(layer "F.Fab")
@@
 		(tags "screw terminal thread redcube thr power connector")
 		(property "Reference" "J4"
-			(at 0 -6 270)
+			(at 0 -6 90)
 			(layer "F.SilkS")
 			(hide yes)
@@
 			)
 		)
-		(property "Value" "Output"
-			(at 0 6 270)
+		(property "Value" "~"
+			(at 0 6 -90)
 			(unlocked yes)
 			(layer "F.SilkS")
+			(hide yes)
 			(effects
 				(font
@@
 			)
 		)
+		(property "Label" "Output"
+			(at 0 6 -90)
+			(unlocked yes)
+			(layer "F.SilkS")
+			(effects
+				(font
+					(size 1 1)
+					(thickness 0.15)
+				)
+			)
+		)
 		(property ki_fp_filters "TerminalBlock*:*")
 		(sheetname "Root")
@@
 		)
 		(fp_text user "${REFERENCE}"
-			(at 0 0 -90)
+			(at 0 0 90)
 			(layer "F.Fab")
 			(effects
@@
 			)
 		)
-		(property "Value" "I2C"
+		(property "Value" "~"
 			(at 0 -6 180)
 			(layer "F.SilkS")
+			(hide yes)
 			(effects
 				(font
@@
 			)
 		)
+		(property "Label" "I2C"
+			(at 0 -6 0)
+			(layer "F.SilkS")
+			(effects
+				(font
+					(size 1 1)
+					(thickness 0.15)
+				)
+			)
+		)
 		(property ki_fp_filters "Connector*:*_1x??-1MP*")
 		(sheetname "Root")
@@
 		(sheetname "Root")
 		(sheetfile "power-monitor.kicad_sch")
-		(attr exclude_from_pos_files)
+		(attr exclude_from_pos_files exclude_from_bom)
 		(fp_circle
 			(center 0 0)
@@
 			)
 		)
-		(property "Value" "PROG"
+		(property "Value" "~"
 			(at 0 -2.3 -90)
 			(layer "F.Fab")
+			(hide yes)
 			(effects
 				(font
@@
 			)
 		)
+		(property "Label" "PROG"
+			(at 0 -2.3 -90)
+			(unlocked yes)
+			(layer "F.SilkS")
+			(effects
+				(font
+					(size 1 1)
+					(thickness 0.15)
+				)
+			)
+		)
 		(property ki_fp_filters "Connector*:*_2x??_*")
 		(sheetname "Root")
 		(sheetfile "power-monitor.kicad_sch")
-		(attr exclude_from_pos_files)
+		(attr exclude_from_pos_files exclude_from_bom)
 		(fp_line
 			(start -1.27 1.27)
