File: hardware/power-monitor.kicad_sch (KiCad schematic)
At the start: 35 parts, among them J1 Input A, J10 I2C, J2 Screw_Terminal_01x06, J3 PROG, J4 Output, J5 Screw_Terminal_01x01, J6 Ground, J7 Input B, J8 Screw_Terminal_01x01, J9 I2C, SW1 RESET, U1 ESP32-C3-WROOM-02-NOTHERMAL, U2 INA228, U4 INA228

Commit message: Improve BOM
Parts:
- C4: value C -> 1uF
- H1, H2, H3, H4: now left out of the parts list
- J1: value Input A -> ~; Label (none) -> Input A
- J10, J9: value I2C -> ~; Label (none) -> I2C
- J3: value PROG -> ~; Label (none) -> PROG; now left out of the parts list
- J4: value Output -> ~; Label (none) -> Output
- J5, J8: value Screw_Terminal_01x01 -> ~
- J6: value Ground -> ~; Label (none) -> Ground
- J7: value Input B -> ~; Label (none) -> Input B
Changed lines of the file:
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@@
 			)
 		)
-		(property "Value" "Screw_Terminal_01x01"
+		(property "Value" "~"
 			(at 184.15 128.27 0)
 			(effects
@@
 			)
 		)
-		(property "Value" "Screw_Terminal_01x01"
+		(property "Value" "~"
 			(at 184.15 133.35 0)
 			(effects
@@
 		(unit 1)
 		(exclude_from_sim no)
-		(in_bom yes)
+		(in_bom no)
 		(on_board yes)
 		(dnp no)
-		(fields_autoplaced yes)
 		(property "Reference" "J3"
 			(at 93.98 135.89 0)
@@
 			)
 		)
-		(property "Value" "PROG"
+		(property "Value" "~"
 			(at 93.98 138.43 0)
 			(effects
@@
 					(size 1.27 1.27)
 				)
+				(hide yes)
 			)
 		)
@@
 			)
 		)
+		(property "Label" "PROG"
+			(at 93.98 138.938 0)
+			(effects
+				(font
+					(size 1.27 1.27)
+				)
+			)
+		)
 		(pin "5"
 		)
@@
 		(unit 1)
 		(exclude_from_sim no)
-		(in_bom yes)
+		(in_bom no)
 		(on_board yes)
 		(dnp no)
@@
 		(on_board yes)
 		(dnp no)
-		(fields_autoplaced yes)
 		(property "Reference" "J9"
 			(at 95.25 178.1555 0)
@@
 			)
 		)
-		(property "Value" "I2C"
+		(property "Value" "~"
 			(at 95.25 180.6955 0)
 			(effects
@@
 				)
 				(justify left)
+				(hide yes)
 			)
 		)
@@
 			)
 		)
+		(property "Label" "I2C"
+			(at 95.25 180.34 0)
+			(effects
+				(font
+					(size 1.27 1.27)
+				)
+				(justify left)
+			)
+		)
 		(pin "4"
 		)
@@
 		(unit 1)
 		(exclude_from_sim no)
-		(in_bom yes)
+		(in_bom no)
 		(on_board yes)
 		(dnp no)
@@
 		(unit 1)
 		(exclude_from_sim no)
-		(in_bom yes)
+		(in_bom no)
 		(on_board yes)
 		(dnp no)
@@
 			)
 		)
-		(property "Value" "Ground"
+		(property "Value" "~"
 			(at 184.15 123.19 0)
 			(effects
@@
 			)
 		)
+		(property "Label" "Ground"
+			(at 184.15 127 0)
+			(effects
+				(font
+					(size 1.27 1.27)
+				)
+				(hide yes)
+			)
+		)
 		(pin "1"
 		)
@@
 			)
 		)
-		(property "Value" "Input A"
+		(property "Value" "~"
 			(at 184.15 104.14 0)
 			(effects
@@
 					(size 1.27 1.27)
 				)
+				(hide yes)
 			)
 		)
@@
 			)
 		)
+		(property "Label" "Input A"
+			(at 184.15 104.902 0)
+			(effects
+				(font
+					(size 1.27 1.27)
+				)
+			)
+		)
 		(pin "1"
 		)
@@
 			)
 		)
-		(property "Value" "I2C"
+		(property "Value" "~"
 			(at 132.08 179.4255 0)
 			(effects
@@
 				)
 				(justify left)
+				(hide yes)
 			)
 		)
@@
 			)
 		)
+		(property "Label" "I2C"
+			(at 132.334 179.578 0)
+			(effects
+				(font
+					(size 1.27 1.27)
+				)
+				(justify left)
+			)
+		)
 		(pin "4"
 		)
@@
 			)
 		)
-		(property "Value" "C"
+		(property "Value" "1uF"
 			(at 36.83 46.9899 0)
 			(effects
@@
 			)
 		)
-		(property "Value" "Input B"
+		(property "Value" "~"
 			(at 184.15 44.45 0)
 			(effects
@@
 					(size 1.27 1.27)
 				)
+				(hide yes)
 			)
 		)
@@
 			)
 		)
+		(property "Label" "Input B"
+			(at 184.15 45.212 0)
+			(effects
+				(font
+					(size 1.27 1.27)
+				)
+			)
+		)
 		(pin "1"
 		)
@@
 			)
 		)
-		(property "Value" "Output"
+		(property "Value" "~"
 			(at 184.15 73.66 0)
 			(effects
@@
 					(size 1.27 1.27)
 				)
+				(hide yes)
 			)
 		)
@@
 			)
 		)
+		(property "Label" "Output"
+			(at 184.15 74.422 0)
+			(effects
+				(font
+					(size 1.27 1.27)
+				)
+			)
+		)
 		(pin "1"
 		)
@@
 		(unit 1)
 		(exclude_from_sim no)
-		(in_bom yes)
+		(in_bom no)
 		(on_board yes)
 		(dnp no)
